Commit message: camera 추가 (xtion_pro)
카메라를 추가해서 points 값 토픽으로 얻는데 성공.
이에 따라, pointCloud2 값을 rviz 상에서 확인했을때, 지형지물을 잘
확인하는것을 보았음.

File: vuasrl_ws/src/tugcar_description/urdf/robot_arm/manipulator_gazebo.xacro (robot description, xacro)
@@ -1,4 +1,6 @@
 <?xml version="1.0"?>
 <robot name="smart_tugcar" xmlns:xacro="http://ros.org/wiki/xacro">
+  <!-- Include xtion_pro Sensors -->
+  <xacro:include filename="$(find tugcar_description)/urdf/sensors/xtion_pro_live.urdf.xacro"/>
   <!-- Gazebo Reference macro -->
   <xacro:macro name="RefLink" params="ref">
@@ -13,4 +15,8 @@
     </gazebo>
   </xacro:macro>
+   <material name="Cam_Color">
+        <color rgba="0.0 0.0 0.75 1.0"/>
+   </material>
+  <xacro:property name="deg_to_rad" value="0.01745329251994329577"/>
   <!-- Link1 -->
   <RefLink ref="link1"/>
@@ -40,4 +46,9 @@
     </plugin>
   </gazebo>
+  <!-- Define RGB-D sensor -->
+  <xacro:xtion_pro_live name="rgbd_camera" parent="base">
+    <origin xyz="-0.06 0.0 0.06" rpy="${0.0 * deg_to_rad} ${360.0 * deg_to_rad} ${0.0 * deg_to_rad}"/>
+    <origin xyz="0 0 0" rpy="${-90 * deg_to_rad} ${0 * deg_to_rad} ${-90 * deg_to_rad}" />
+  </xacro:xtion_pro_live>
   <gazebo>
     <!-- loading plugin: mimic joints works in gazebo now -->

Commit message: Resolved merge conflicts

File: vuasrl_ws/src/tugcar_description/urdf/robot_arm/manipulator_gazebo.xacro (robot description, xacro)
@@ -1,4 +1,6 @@
 <?xml version="1.0"?>
 <robot name="smart_tugcar" xmlns:xacro="http://ros.org/wiki/xacro">
+  <!-- Include xtion_pro Sensors -->
+  <xacro:include filename="$(find tugcar_description)/urdf/sensors/xtion_pro_live.urdf.xacro"/>
   <!-- Gazebo Reference macro -->
   <xacro:macro name="RefLink" params="ref">
@@ -13,4 +15,8 @@
     </gazebo>
   </xacro:macro>
+   <material name="Cam_Color">
+        <color rgba="0.0 0.0 0.75 1.0"/>
+   </material>
+  <xacro:property name="deg_to_rad" value="0.01745329251994329577"/>
   <!-- Link1 -->
   <RefLink ref="link1"/>
@@ -40,4 +46,9 @@
     </plugin>
   </gazebo>
+  <!-- Define RGB-D sensor -->
+  <xacro:xtion_pro_live name="mani_camera" parent="base">
+    <origin xyz="-0.06 0.0 0.06" rpy="${0.0 * deg_to_rad} ${360.0 * deg_to_rad} ${0.0 * deg_to_rad}"/>
+    <origin xyz="0 0 0" rpy="${-90 * deg_to_rad} ${0 * deg_to_rad} ${-90 * deg_to_rad}" />
+  </xacro:xtion_pro_live>
   <gazebo>
     <!-- loading plugin: mimic joints works in gazebo now -->
