Commit message: Adding FAST_LIO files

File: vuasrl_ws/src/vuasrl_arm_description/urdf/vuasrl_arm.xacro (robot description, xacro)
@@ -1,245 +1,209 @@
-<?xml version="1.0"?>
-<!-- Open_Manipulator Chain -->
-<robot xmlns:xacro="http://ros.org/wiki/xacro">
-  <!-- Link 1 -->
-  <link name="link1">
-    <visual>
-      <origin xyz="0 0 0" rpy="0 0 0"/>
-      <geometry>
-        <mesh filename="package://open_manipulator_description/meshes/chain_link1.stl" scale="0.001 0.001 0.001"/>
-      </geometry>
-      <material name="grey"/>
+<?xml version="1.0" ?>
+<robot xmlns:xacro="http://www.ros.org/wiki/xacro">
+<link name="link1">
+  <inertial>
+    <origin xyz="0.0001816853136070254 -2.1915878376977466e-17 0.020129887613482035" rpy="0 0 0"/>
+    <mass value="7.9119962e-02"/>
+    <inertia ixx="0.002145" iyy="0.004951" izz="0.006213" ixy="-0.0" iyz="-0.0" ixz="-1.3e-05"/>
+  </inertial>
+  <visual>
+    <origin xyz="0 0 0" rpy="0 0 0"/>
+    <geometry>
+      <mesh filename="package://vuasrl_arm_description/meshes/base_link.stl" scale="0.001 0.001 0.001"/>
+    </geometry>
+    <material name="silver"/>
+  </visual>
+  <collision>
+    <origin xyz="0 0 0" rpy="0 0 0"/>
+    <geometry>
+      <mesh filename="package://vuasrl_arm_description/meshes/base_link.stl" scale="0.001 0.001 0.001"/>
+    </geometry>
+  </collision>
+</link>
+<link name="link2">
+  <inertial>
+    <origin xyz="-2.328586629074536e-11 -2.8877387782838815e-10 0.020681716416087625" rpy="0 0 0"/>
+    <mass value="9.8406837e-02"/>
+    <inertia ixx="0.000355" iyy="0.00039" izz="0.000302" ixy="0.0" iyz="-0.0" ixz="0.0"/>
+  </inertial>
+  <visual>
+    <origin xyz="-0.03 -0.0 -0.048" rpy="0 0 0"/>
+    <geometry>
+      <mesh filename="package://vuasrl_arm_description/meshes/link1_1.stl" scale="0.001 0.001 0.001"/>
+    </geometry>
+    <material name="silver"/>
+  </visual>
+  <collision>
+    <origin xyz="-0.03 -0.0 -0.048" rpy="0 0 0"/>
+    <geometry>
+      <mesh filename="package://vuasrl_arm_description/meshes/link1_1.stl" scale="0.001 0.001 0.001"/>
+    </geometry>
+  </collision>
+</link>
+<link name="link3">
+  <inertial>
+    <origin xyz="-0.004542317857195898 0.0005782036806908492 0.09874905854464662" rpy="0 0 0"/>
+    <mass value="1.3850917e-01"/>
+    <inertia ixx="0.009439" iyy="0.009407" izz="0.0009" ixy="-1e-06" iyz="1.5e-05" ixz="0.000653"/>
+  </inertial>
+  <visual>
+    <origin xyz="-0.03 -0.0 -0.078" rpy="0 0 0"/>
+    <geometry>
+      <mesh filename="package://vuasrl_arm_description/meshes/link2_1.stl" scale="0.001 0.001 0.001"/>
+    </geometry>
+    <material name="silver"/>
+  </visual>
+  <collision>
+    <origin xyz="-0.03 -0.0 -0.078" rpy="0 0 0"/>
+    <geometry>
+      <mesh filename="package://vuasrl_arm_description/meshes/link2_1.stl" scale="0.001 0.001 0.001"/>
+    </geometry>
+  </collision>
+</link>
+<link name="link4">
+  <inertial>
+    <origin xyz="4.336808689942018e-18 0.0005787515631340847 0.10231346303330496" rpy="0 0 0"/>
+    <mass value="1.3274562e-01"/>
+    <inertia ixx="0.010801" iyy="0.010515" izz="0.000691" ixy="0.0" iyz="1.6e-05" ixz="0.0"/>
+  </inertial>
+  <visual>
+    <origin xyz="-0.005 -0.0005 -0.243" rpy="0 0 0"/>
+    <geometry>
+      <mesh filename="package://vuasrl_arm_description/meshes/link3_1.stl" scale="0.001 0.001 0.001"/>
+    </geometry>
+    <material name="silver"/>
+  </visual>
+  <collision>
+    <origin xyz="-0.005 -0.0005 -0.243" rpy="0 0 0"/>
+    <geometry>
+      <mesh filename="package://vuasrl_arm_description/meshes/link3_1.stl" scale="0.001 0.001 0.001"/>
+    </geometry>
+  </collision>
+</link>
+<link name="link5">
+  <inertial>
+    <origin xyz="2.8536201179818477e-16 -5.72784007724092e-15 0.04451102048440414" rpy="0 0 0"/>
+    <mass value="1.4327573e-01"/>
+    <inertia ixx="0.00218" iyy="0.00154" izz="0.000828" ixy="-0.0" iyz="0.0" ixz="-0.0"/>
+  </inertial>
+  <visual>
+    <origin xyz="-0.005 -0.001 -0.433" rpy="0 0 0"/>
+    <geometry>
+      <mesh filename="package://vuasrl_arm_description/meshes/link4_1.stl" scale="0.001 0.001 0.001"/>
+    </geometry>
+    <material name="silver"/>
+  </visual>
+  <collision>
+    <origin xyz="-0.005 -0.001 -0.433" rpy="0 0 0"/>
+    <geometry>
+      <mesh filename="package://vuasrl_arm_description/meshes/link4_1.stl" scale="0.001 0.001 0.001"/>
+    </geometry>
+  </collision>
+</link>
+<link name="link_grip_r">
+  <inertial>
+    <origin xyz="0 0 0" rpy="0 0 0"/>
+    <mass value="1.0e-03"/>
+    <inertia ixx="1.0e-03" iyy="1.0e-03" izz="1.0e-03" ixy="0.0" iyz="0.0" ixz="0.0"/>
+  </inertial>
+  <visual>
+    <origin xyz="-0.01 0.033 -0.95715" rpy="0 0 0"/>
+    <geometry>
+      <mesh filename="package://vuasrl_arm_description/meshes/link_grip_r_1.stl" scale="0.001 0.001 0.001"/>
+    </geometry>
+    <material name="silver"/>
+  </visual>
+  <collision>
+    <origin xyz="-0.01 0.033 -0.95715" rpy="0 0 0"/>
+    <geometry>
+      <mesh filename="package://vuasrl_arm_description/meshes/link_grip_r_1.stl" scale="0.001 0.001 0.001"/>
+    </geometry>
+  </collision>
+</link>
+<link name="link_grip_l">
+  <inertial>
+    <origin xyz="0 0 0" rpy="0 0 0"/>
+    <mass value="1.0e-03"/>
+    <inertia ixx="1.0e-03" iyy="1.0e-03" izz="1.0e-03" ixy="0.0" iyz="0.0" ixz="0.0"/>
+  </inertial>
+  <visual>
+    <origin xyz="-0.01 -0.037 -0.95715" rpy="0 0 0"/>
+    <geometry>
+      <mesh filename="package://vuasrl_arm_description/meshes/link_grip_l_1.stl" scale="0.001 0.001 0.001"/>
+    </geometry>
+    <material name="silver"/>
+  </visual>
+  <collision>
+    <origin xyz="-0.01 -0.037 -0.95715" rpy="0 0 0"/>
+    <geometry>
+      <mesh filename="package://vuasrl_arm_description/meshes/link_grip_l_1.stl" scale="0.001 0.001 0.001"/>
+    </geometry>
+  </collision>
+</link>
+<joint name="joint1" type="revolute">
+  <origin xyz="0.03 0.0 0.048" rpy="0 0 0"/>
+  <parent link="link1"/>
+  <child link="link2"/>
+  <axis xyz="0.0 0.0 1.0"/>
+  <limit velocity="4.8" effort="1" lower="${-pi*0.9}" upper="${pi*0.9}" />
+</joint>
+<joint name="joint2" type="revolute">
+  <origin xyz="0.0 0.0 0.03" rpy="0 0 0"/>
+  <parent link="link2"/>
+  <child link="link3"/>
+  <axis xyz="0.0 1.0 0.0"/>
+  <limit velocity="4.8" effort="1" lower="${-pi*0.57}" upper="${pi*0.5}" />
+</joint>
+<joint name="joint3" type="revolute">
+  <origin xyz="-0.025 0.0005 0.165" rpy="0 0 0"/>
+  <parent link="link3"/>
+  <child link="link4"/>
+  <axis xyz="0.0 1.0 0.0"/>
+  <limit velocity="4.8" effort="1" lower="${-pi*0.3}" upper="${pi*0.44}" />
+</joint>
+<joint name="joint4" type="revolute">
+  <origin xyz="0.0 0.0005 0.19" rpy="0 0 0"/>
+  <parent link="link4"/>
+  <child link="link5"/>
+  <axis xyz="0.0 1.0 0.0"/>
+  <limit velocity="4.8" effort="1" lower="${-pi*0.57}" upper="${pi*0.65}" />
+</joint>
+<joint name="grip_joint" type="prismatic">
+  <origin xyz="0.005 -0.034 0.52415" rpy="0 0 0"/>
+  <parent link="link5"/>
+  <child link="link_grip_r"/>
+  <axis xyz="0.0 1.0 0.0"/>
+  <limit velocity="4.8" effort="1" lower="-0.010" upper="0.019" />
+</joint>
+<joint name="grip_joint_sub" type="prismatic">
+  <origin xyz="0.005 0.036 0.52415" rpy="0 0 0"/>
+  <parent link="link5"/>
+  <child link="link_grip_l"/>
+  <axis xyz="0.0 -1.0 0.0"/>
+  <limit velocity="4.8" effort="1" lower="-0.010" upper="0.019" />
+  <mimic joint="grip_joint" multiplier="1"/>
+</joint>
+<!-- end effector joint -->
+<joint name="end_effector_joint" type="fixed">
+  <origin xyz="0.0 0.0 0.115" rpy="0 0 0"/>
+  <parent link="link5"/>
+  <child link="end_effector_link"/>
+</joint>
+<!-- end effector link -->
+<link name="end_effector_link">
+  <visual>
+    <origin xyz="0 0 0" rpy="0 0 0"/>
+    <geometry>
+      <box size="0.01 0.01 0.01" />
+    </geometry>
+    <material name="red"/>
     </visual>
-    <collision>
-      <origin xyz="0 0 0" rpy="0 0 0"/>
-      <geometry>
-        <mesh filename="package://open_manipulator_description/meshes/chain_link1.stl" scale="0.001 0.001 0.001"/>
-      </geometry>
-    </collision>
-    <inertial>
-      <origin xyz="3.0876154e-04 0.0000000e+00 -1.2176461e-04" />
-      <mass value="7.9119962e-02" />
-      <inertia ixx="1.2505234e-05" ixy="0.0" ixz="-1.7855208e-07"
-               iyy="2.1898364e-05" iyz="0.0"
-               izz="1.9267361e-05" />
-    </inertial>
-  </link>
-  <!-- Joint 1 -->
-  <joint name="joint1" type="revolute">
-    <parent link="link1"/>
-    <child link="link2"/>
-    <origin xyz="0.012 0.0 0.017" rpy="0 0 0"/>
-    <axis xyz="0 0 1"/>
-    <limit velocity="4.8" effort="1" lower="${-pi*0.9}" upper="${pi*0.9}" />
-  </joint>
-  <!--  Link 2 -->
-  <link name="link2">
-    <visual>
-      <origin xyz="0 0 0.019" rpy="0 0 0"/>
-      <geometry>
-        <mesh filename="package://open_manipulator_description/meshes/chain_link2.stl" scale="0.001 0.001 0.001"/>
-      </geometry>
-      <material name="grey"/>
-    </visual>
-    <collision>
-      <origin xyz="0 0 0.019" rpy="0 0 0"/>
-      <geometry>
-        <mesh filename="package://open_manipulator_description/meshes/chain_link2.stl" scale="0.001 0.001 0.001"/>
-      </geometry>
-    </collision>
-    <inertial>
-      <origin xyz="-3.0184870e-04 5.4043684e-04 ${0.018 + 2.9433464e-02}" />
-      <mass value="9.8406837e-02" />
-      <inertia ixx="3.4543422e-05" ixy="-1.6031095e-08" ixz="-3.8375155e-07"
-               iyy="3.2689329e-05" iyz="2.8511935e-08"
-               izz="1.8850320e-05" />
-    </inertial>
-  </link>
-  <!--  Joint 2 -->
-  <joint name="joint2" type="revolute">
-    <parent link="link2"/>
-    <child link="link3"/>
-    <origin xyz="0.0 0.0 0.0595" rpy="0 0 0"/>
-    <axis xyz="0 1 0"/>
-    <limit velocity="4.8" effort="1" lower="${-pi*0.57}" upper="${pi*0.5}" />
-  </joint>
-  <!--  Link 3 -->
-  <link name="link3">
-    <visual>
-      <origin xyz="0 0 0" rpy="0 0 0"/>
-      <geometry>
-        <mesh filename="package://open_manipulator_description/meshes/chain_link3.stl" scale="0.001 0.001 0.001"/>
-      </geometry>
-      <material name="grey"/>
-    </visual>
-    <collision>
-      <origin xyz="0 0 0" rpy="0 0 0"/>
-      <geometry>
-        <mesh filename="package://open_manipulator_description/meshes/chain_link3.stl" scale="0.001 0.001 0.001"/>
-      </geometry>
-    </collision>
-    <inertial>
-      <origin xyz="1.0308393e-02 3.7743363e-04 1.0170197e-01" />
-      <mass value="1.3850917e-01" />
-      <inertia ixx="3.3055381e-04" ixy="-9.7940978e-08" ixz="-3.8505711e-05"
-               iyy="3.4290447e-04" iyz="-1.5717516e-06"
-               izz="6.0346498e-05" />
-    </inertial>
-  </link>
-  <!--  Joint 3 -->
-  <joint name="joint3" type="revolute">
-    <parent link="link3"/>
-    <child link="link4"/>
-    <origin xyz="0.024 0 0.128" rpy="0 0 0"/>
-    <axis xyz="0 1 0"/>
-    <limit velocity="4.8" effort="1" lower="${-pi*0.3}" upper="${pi*0.44}" />
-  </joint>
-  <!--  Link 4 -->
-  <link name="link4">
-    <visual>
-      <origin xyz="0 0 0" rpy="0 0 0"/>
-      <geometry>
-        <mesh filename="package://open_manipulator_description/meshes/chain_link4.stl" scale="0.001 0.001 0.001"/>
-      </geometry>
-      <material name="grey"/>
-    </visual>
-    <collision>
-      <origin xyz="0 0 0" rpy="0 0 0"/>
-      <geometry>
-        <mesh filename="package://open_manipulator_description/meshes/chain_link4.stl" scale="0.001 0.001 0.001"/>
-      </geometry>
-    </collision>
-    <inertial>
-      <origin xyz="9.0909590e-02 3.8929816e-04 2.2413279e-04" />
-      <mass value="1.3274562e-01" />
-      <inertia ixx="3.0654178e-05" ixy="-1.2764155e-06" ixz="-2.6874417e-07"
-               iyy="2.4230292e-04" iyz="1.1559550e-08"
-               izz="2.5155057e-04" />
-    </inertial>
-  </link>
-  <!--  Joint 4 -->
-  <joint name="joint4" type="revolute">
-    <parent link="link4"/>
-    <child link="link5"/>
-    <origin xyz="0.124 0.0 0.0" rpy="0 0 0"/>
-    <axis xyz="0 1 0"/>
-    <limit velocity="4.8" effort="1" lower="${-pi*0.57}" upper="${pi*0.65}" />
-  </joint>
-  <!--  Link 5 -->
-  <link name="link5">
-    <visual>
-      <origin xyz="0 0 0" rpy="0 0 0"/>
-      <geometry>
-        <mesh filename="package://open_manipulator_description/meshes/chain_link5.stl" scale="0.001 0.001 0.001"/>
-      </geometry>
-      <material name="grey"/>
-    </visual>
-    <collision>
-      <origin xyz="0 0 0" rpy="0 0 0"/>
-      <geometry>
-        <mesh filename="package://open_manipulator_description/meshes/chain_link5.stl" scale="0.001 0.001 0.001"/>
-      </geometry>
-    </collision>
-    <inertial>
-      <origin xyz="4.4206755e-02 3.6839985e-07 8.9142216e-03" />
-      <mass value="1.4327573e-01" />
-      <inertia ixx="8.0870749e-05" ixy="0.0" ixz="-1.0157896e-06"
-               iyy="7.5980465e-05" iyz="0.0"
-               izz="9.3127351e-05" />
-    </inertial>
-  </link>
-  <!--  Gripper joint -->
-  <joint name="gripper" type="prismatic">
-    <parent link="link5"/>
-    <child link="gripper_link"/>
-    <origin xyz="0.0817 0.021 0.0" rpy="0 0 0"/>
-    <axis xyz="0 1 0"/>
-    <limit velocity="4.8" effort="1" lower="-0.010" upper="0.019" />
-  </joint>
-  <!--  Gripper link -->
-  <link name="gripper_link">
-    <visual>
-      <origin xyz="0.0 0.0 0" rpy="0 0 0"/>
-      <geometry>
-        <mesh filename="package://open_manipulator_description/meshes/chain_link_grip_l.stl" scale="0.001 0.001 0.001"/>
-      </geometry>
-      <material name="grey"/>
-    </visual>
-    <collision>
-      <origin xyz="0.0 0.0 0" rpy="0 0 0"/>
-      <geometry>
-        <mesh filename="package://open_manipulator_description/meshes/chain_link_grip_l.stl" scale="0.001 0.001 0.001"/>
-      </geometry>
-    </collision>
-    <inertial>
-      <origin xyz="0 0 0" />
-      <mass value="1.0e-03" />
-      <inertia ixx="1.0e-03" ixy="0.0" ixz="0.0"
-               iyy="1.0e-03" iyz="0.0"
-               izz="1.0e-03" />
-    </inertial>
-  </link>
-  <!--  Gripper joint sub -->
-  <joint name="gripper_sub" type="prismatic">
-    <parent link="link5"/>
-    <child link="gripper_link_sub"/>
-    <origin xyz="0.0817 -0.021 0" rpy="0 0 0"/>
-    <axis xyz="0 -1 0"/>
-    <limit velocity="4.8" effort="1" lower="-0.010" upper="0.019" />
-    <mimic joint="gripper" multiplier="1"/>
-  </joint>
-  <!--  Gripper link sub -->
-  <link name="gripper_link_sub">
-    <visual>
-      <origin xyz="0.0 -0.0 0" rpy="0 0 0"/>
-      <geometry>
-        <mesh filename="package://open_manipulator_description/meshes/chain_link_grip_r.stl" scale="0.001 0.001 0.001"/>
-      </geometry>
-      <material name="grey"/>
-    </visual>
-    <collision>
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
File: vuasrl_ws/src/vuasrl_car_description/urdf/vuasrl_car.xacro (robot description, xacro)
@@ -1,4 +1,4 @@
 <?xml version="1.0" ?>
-<robot name="vuasrl_car" xmlns:xacro="http://www.ros.org/wiki/xacro">
+<robot name="vuasrl_manipulation" xmlns:xacro="http://www.ros.org/wiki/xacro">
 <xacro:include filename="$(find vuasrl_car_description)/urdf/materials.xacro" />
 <xacro:include filename="$(find vuasrl_car_description)/urdf/vuasrl_car.trans" />
@@ -9,5 +9,5 @@
     <origin xyz="-0.0024815786222996896 8.508916291582655e-12 0.0794086767825376" rpy="0 0 0"/>
     <mass value="4.692054269661653"/>
-    <inertia ixx="0.016864" iyy="0.034752" izz="0.046313" ixy="-0.0" iyz="0.0" ixz="0.000383"/>
+    <inertia ixx="0.016864" iyy="0.034781" izz="0.046341" ixy="0.0" iyz="0.0" ixz="-0.000207"/>
   </inertial>
   <visual>
@@ -134,5 +134,5 @@
       <origin xyz="0 0 0" rpy="0 0 0"/>
       <geometry>
-        <box size ="0.04 0.02 0.01"/>
+        <box size ="0.01 0.02 0.01"/>
       </geometry>
       <material name="white"/>
@@ -140,5 +140,5 @@
   <collision>
       <geometry>
-        <box size = "0.04 0.02 0.01"/>
+        <box size = "0.01 0.02 0.01"/>
       </geometry>
   </collision>
@@ -174,5 +174,5 @@
 </joint>
 <joint name="lidar_base" type="fixed">
-  <origin xyz="-0.17 0.0 0.30" rpy="0 0 0"/>
+  <origin xyz="0.0 0.0 0.30" rpy="0 0 0"/>
   <parent link="base_link"/>
   <child link="ouster_link"/>
@@ -181,5 +181,5 @@
   <parent link="base_link"/>
   <child link="imu_link"/>
-  <origin xyz="-0.03 0 0.125" rpy="0 0 0"/>
+  <origin xyz="0.03 0 0.125" rpy="0 0 0"/>
 </joint>
 </robot>
